File: Eagle PCB Design Files/Ebike_Project/Arduino_Shield_6_5_19_REV3.sch (EAGLE design)
At the start: 0 parts

Commit message: Completed REV3 of board
REV adds a larger DC/DC converter and connector for a 12V headlight
Other:
- note added: "36-72V/12V DCDC"
- note added: "BMS_SWITCH"
- note added: "Connector Crimp Series 70058 - Part No: 16020086"
- note added: "Connector Housing Series 70543 - Part No: 7054300XX"
- note added: "Connector Plug Series 70066 - Part No: 505794XX"
- note added: "IGNITION_SWITCH"
- note added: "Wire to Wire Housing Crimp: 70021-1021"
- note added: "Wire to Wire Housing Series: 70107 - Part No: 701070003"

Commit message: Completed REV3
REV3 is identical to REV4 but uses an off the shelf arduino nano.
Parts:
- added CXTR_BMS, CXTR_DASH: 4PIN_.1"_CONNECTOR, EBike_Project_Library:4PIN_.1"_CONNECTOR
- added CXTR_HALL_SENSOR: 3PIN_.1"_CONNECTOR, EBike_Project_Library:3PIN_.1"_CONNECTOR
- added CXTR_HEADLIGHT, CXTR_POWER: 2PIN_.1"_CONNECTOR, EBike_Project_Library:2PIN_.1"_CONNECTOR
- added R1: 4.99, EBike_Project_Library:RESISTOR_4.99K_0805-0805-1/8W-1%
- added U$2: SKM15C-12_DCDC, EBike_Project_Library:SKM15C-12_DCDC
- added U$3: ARDUINO_NANO, EBike_Project_Library:ARDUINO_NANO
Connections:
- new net +12V: CXTR_HEADLIGHT.2, U$2.+VOUT, U$3.RAW
- new net +5V: CXTR_DASH.2, CXTR_HALL_SENSOR.1, R1.2, U$3.5.5V
- new net B+: CXTR_POWER.2, U$2.+VIN
- new net B-_ECU: CXTR_BMS.4, CXTR_DASH.1, CXTR_HALL_SENSOR.3, CXTR_HEADLIGHT.1, CXTR_POWER.1, U$2.-VIN, U$2.-VOUT, U$3.GND
- new net D2_HALL: CXTR_HALL_SENSOR.2, R1.1, U$3.D2
- new net LCD_SCL_A5: CXTR_DASH.3, U$3.A5
- new net LCD_SDA_A4: CXTR_DASH.4, U$3.A4
- new net RX_NANO_D10: CXTR_BMS.3, U$3.D10
- new net TX_NANO_D11: CXTR_BMS.2, U$3.D11
Other:
- note added: "CONNECTORS"
- note added: "Connector Housing Series 70543 - Part No: 705430004 (4 PIN)"
- note removed: "Connector Housing Series 70543 - Part No: 7054300XX"
